File: KiCadProject/OptionalOuterUSB/OuterUSB.kicad_sch (KiCad schematic)
At the start: 6 parts, among them J101 USB-C-2.0, J102 Power connector, J103 Data connector, J104 CC connector

Commit message: Made ready to order PCBs. Some problems with ordering due to misunderstanding. Thinking about solutions
Signed-off-by: Eldalote.Electronics <Eldalote.Electronics@gmail.com>
Other:
- company: (none) -> Eldalote Electronics
- title: (none) -> Optional External USB-C connector
Changed lines of the file:
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@@
 (kicad_sch (version 20211123) (generator eeschema)
   (paper "A4")
+  (title_block
+    (title "Optional External USB-C connector")
+    (date "2023-02-02")
+    (rev "0.1")
+    (company "Eldalote Electronics")
+    (comment 2 "Part of the Dive Lamp design")
+  )
   (junction (at 139.7 107.95) (diameter 0) (color 0 0 0 0)
   )
