File: KiCadProject/OptionalOuterUSB/OuterUSB.kicad_pcb (KiCad board)
At the start: 6 copper layers, 13 x 10.3 mm, 6 parts, among them J101 USB-C-2.0, J102 Power connector, J103 Data connector, J104 CC connector

Commit message: Started work on body 3d work
Signed-off-by: Eldalote.Electronics <Eldalote.Electronics@gmail.com>
Parts:
- moved J102 0.80 mm to (148.7, 96.6)
- moved J104 0.21 mm to (144.5, 98.0)
- moved J103 0.07 mm to (155.5, 98.0)
Routing:
- net /CC1: track 6.79 -> 8.83 mm
- net GND: track 9.53 -> 7.60 mm, vias 8 -> 9
- net /CC2: track 10.5 -> 9.20 mm
- net /Data+: track 10.3 -> 11.0 mm
- added copper zone on In2.Cu, net GND
- removed copper zone on In3.Cu, net GND
Other:
- copper layers 6 -> 4
- board text added: "Jeremy"
