File: KiCadProject/BatteryManagementBoard/BatteryManagementBoard.kicad_pcb (KiCad board)
At the start: 6 copper layers, 45 x 45 mm, 93 parts, among them J201 USB-C-2.0, J202 XT30, J203 Conn_02x05, J204 XT60, J205 Conn_02x05, J206 Conn_01x02_Male, J207 Conn_01x05_Male, J208 JST_B5B_XH, J209 Optional off board USB power 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, J210 Optional off board USB CC con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, Q301 NFET_Gatenames, Q302 NFET_Gatenames, Q303 NFET_Gatenames, Q304 NFET_Gatenames, Q305 PMOS_Gatenames, U301 BQ25713, U401 AP63205WU, U402 SC189, U501 PTN5150

Commit message: Started work on body 3d work
Signed-off-by: Eldalote.Electronics <Eldalote.Electronics@gmail.com>
Changed lines of the file:
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@@
       (usegerberattributes true)
       (usegerberadvancedattributes false)
-      (creategerberjobfile false)
+      (creategerberjobfile true)
       (svguseinch false)
       (svgprecision 6)
@@
   (via (at 152.6 92) (size 0.45) (drill 0.2) (layers "F.Cu" "B.Cu") (net 2))
   (via (at 163.3 93.2) (size 0.45) (drill 0.2) (layers "F.Cu" "B.Cu") (net 2))
-  (via (at 137.1 107.4) (size 0.45) (drill 0.2) (layers "F.Cu" "B.Cu") (free) (net 2))
+  (via (at 137.1 107.3) (size 0.45) (drill 0.2) (layers "F.Cu" "B.Cu") (free) (net 2))
   (via (at 149 94) (size 0.45) (drill 0.2) (layers "F.Cu" "B.Cu") (net 2))
   (via (at 132 94.1) (size 0.45) (drill 0.2) (layers "F.Cu" "B.Cu") (net 2))
@@
         (xy 133.7 107.7)
         (xy 133.4 108)
-        (xy 133.4 110.8)
-        (xy 130.6 110.8)
-        (xy 129.4 107.8)
-        (xy 133.2 106.4)
-        (xy 133.2 103.8)
-        (xy 135 103.8)
+        (xy 133.4 110.4)
+        (xy 133 110.8)
+        (xy 130.3 110.8)
+        (xy 129.5 109.4)
+        (xy 128.7 107.3)
+        (xy 131.8 107.3)
+        (xy 133.2 105.9)
+        (xy 133.2 104)
+        (xy 133.4 103.8)
+        (xy 134.8 103.8)
+        (xy 135 104)
       )
     )
@@
     (polygon
       (pts
-        (xy 137.1 103.5)
-        (xy 137.1 104.9)
-        (xy 138.6 105.9)
+        (xy 137.3 103.5)
+        (xy 137.3 104.9)
+        (xy 138.6 106.2)
         (xy 138.6 107.3)
         (xy 137.9 108)
@@
         (xy 136.2 108)
         (xy 135.4 107.3)
-        (xy 135.4 103.9)
+        (xy 135.4 104)
         (xy 134.7 103.2)
-        (xy 134.7 99.5)
-        (xy 136.4 99.5)
-        (xy 136.4 102.8)
+        (xy 134.7 99.7)
+        (xy 134.9 99.5)
+        (xy 136.1 99.5)
+        (xy 136.4 99.8)
+        (xy 136.4 102.6)
       )
     )
@@
         (xy 135.1 107.8)
         (xy 137.3 107.8)
-        (xy 137.3 109.3)
-        (xy 134.2 109.2)
-        (xy 133.7 108.6)
-        (xy 132.7 108.5)
-        (xy 132.7 107.5)
-        (xy 134.7 107.5)
+        (xy 137.3 109.2)
+        (xy 134.4 109.2)
+        (xy 133.7 108.5)
+        (xy 132.8 108.5)
+        (xy 132.7 108.4)
+        (xy 132.7 107.6)
+        (xy 132.8 107.5)
+        (xy 134.8 107.5)
       )
     )
@@
         (xy 131.4 90.4)
         (xy 131.4 89)
+        (xy 132.3 87.4)
         (xy 133.8 86.6)
         (xy 135 86.6)
@@
         (xy 131.9 110.9)
         (xy 130.4 110.9)
-        (xy 129.3 107.9)
+        (xy 129.310882 108.794371)
+        (xy 128.7 107.6)
         (xy 129.9 107.6)
         (xy 131.9 107.6)
