File: KiCadProject/SamsungLedBoard/SamsungLedBoard.kicad_pcb (KiCad board)
At the start: 6 copper layers, 45 x 45 mm, 14 parts, among them J1 XT30

Commit message: Started work on body 3d work
Signed-off-by: Eldalote.Electronics <Eldalote.Electronics@gmail.com>
Routing:
- removed copper zone on In1.Cu, net /L1-2
- removed copper zone on In2.Cu, net /L1-2
- removed copper zone on In3.Cu, net /L1-2
- removed copper zone on In4.Cu, net /L1-2
- removed copper zone on In1.Cu, net /L10C
- removed copper zone on In2.Cu, net /L10C
- removed copper zone on In3.Cu, net /L10C
- removed copper zone on In4.Cu, net /L10C
- removed copper zone on In1.Cu, net /L1A
- removed copper zone on In2.Cu, net /L1A
- removed copper zone on In3.Cu, net /L1A
- removed copper zone on In4.Cu, net /L1A
- removed copper zone on In1.Cu, net /L2-3
- removed copper zone on In2.Cu, net /L2-3
- removed copper zone on In3.Cu, net /L2-3
- removed copper zone on In4.Cu, net /L2-3
- removed copper zone on In1.Cu, net /L3-4
- removed copper zone on In2.Cu, net /L3-4
- removed copper zone on In3.Cu, net /L3-4
- removed copper zone on In4.Cu, net /L3-4
- removed copper zone on In1.Cu, net /L4-5
- removed copper zone on In2.Cu, net /L4-5
- removed copper zone on In3.Cu, net /L4-5
- removed copper zone on In4.Cu, net /L4-5
- removed copper zone on In1.Cu, net /L5-6
- removed copper zone on In2.Cu, net /L5-6
- removed copper zone on In3.Cu, net /L5-6
- removed copper zone on In4.Cu, net /L5-6
- removed copper zone on In1.Cu, net /L6-7
- removed copper zone on In2.Cu, net /L6-7
- removed copper zone on In3.Cu, net /L6-7
- removed copper zone on In4.Cu, net /L6-7
- removed copper zone on In1.Cu, net /L7-8
- removed copper zone on In2.Cu, net /L7-8
- removed copper zone on In3.Cu, net /L7-8
- removed copper zone on In4.Cu, net /L7-8
- removed copper zone on In1.Cu, net /L8-9
- removed copper zone on In2.Cu, net /L8-9
- removed copper zone on In3.Cu, net /L8-9
- removed copper zone on In4.Cu, net /L8-9
- removed copper zone on In1.Cu, net /L9-10
- removed copper zone on In2.Cu, net /L9-10
- removed copper zone on In3.Cu, net /L9-10
- removed copper zone on In4.Cu, net /L9-10
Other:
- copper layers 6 -> 2
Changed lines of the file:
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@@
   (layers
     (0 "F.Cu" signal)
-    (1 "In1.Cu" signal)
-    (2 "In2.Cu" signal)
-    (3 "In3.Cu" signal)
-    (4 "In4.Cu" signal)
     (31 "B.Cu" signal)
     (32 "B.Adhes" user "B.Adhesive")
@@
       (layer "F.Mask" (type "Top Solder Mask") (thickness 0.01))
       (layer "F.Cu" (type "copper") (thickness 0.035))
-      (layer "dielectric 1" (type "core") (thickness 0.274) (material "FR4") (epsilon_r 4.5) (loss_tangent 0.02))
-      (layer "In1.Cu" (type "copper") (thickness 0.035))
-      (layer "dielectric 2" (type "prepreg") (thickness 0.274) (material "FR4") (epsilon_r 4.5) (loss_tangent 0.02))
-      (layer "In2.Cu" (type "copper") (thickness 0.035))
-      (layer "dielectric 3" (type "core") (thickness 0.274) (material "FR4") (epsilon_r 4.5) (loss_tangent 0.02))
-      (layer "In3.Cu" (type "copper") (thickness 0.035))
-      (layer "dielectric 4" (type "prepreg") (thickness 0.274) (material "FR4") (epsilon_r 4.5) (loss_tangent 0.02))
-      (layer "In4.Cu" (type "copper") (thickness 0.035))
-      (layer "dielectric 5" (type "core") (thickness 0.274) (material "FR4") (epsilon_r 4.5) (loss_tangent 0.02))
+      (layer "dielectric 1" (type "core") (thickness 1.51) (material "FR4") (epsilon_r 4.5) (loss_tangent 0.02))
       (layer "B.Cu" (type "copper") (thickness 0.035))
       (layer "B.Mask" (type "Bottom Solder Mask") (thickness 0.01))
@@
   (via (at 153.4 99) (size 0.8) (drill 0.4) (layers "F.Cu" "B.Cu") (free) (net 11))
   (via (at 153.4 101.4) (size 0.8) (drill 0.4) (layers "F.Cu" "B.Cu") (free) (net 11))
-  (zone (net 4) (net_name "/L3-4") (layers "F.Cu" "In1.Cu" "In2.Cu" "In3.Cu" "In4.Cu" "B.Cu") (hatch edge 0.508)
+  (zone (net 4) (net_name "/L3-4") (layers F&B.Cu) (hatch edge 0.508)
     (connect_pads yes (clearance 0.2))
     (min_thickness 0.2) (filled_areas_thickness no)
@@
     )
   )
-  (zone (net 9) (net_name "/L8-9") (layers "F.Cu" "In1.Cu" "In2.Cu" "In3.Cu" "In4.Cu" "B.Cu") (hatch edge 0.508)
+  (zone (net 9) (net_name "/L8-9") (layers F&B.Cu) (hatch edge 0.508)
     (connect_pads yes (clearance 0.2))
     (min_thickness 0.2) (filled_areas_thickness no)
@@
     )
   )
-  (zone (net 8) (net_name "/L7-8") (layers "F.Cu" "In1.Cu" "In2.Cu" "In3.Cu" "In4.Cu" "B.Cu") (hatch edge 0.508)
+  (zone (net 8) (net_name "/L7-8") (layers F&B.Cu) (hatch edge 0.508)
     (connect_pads yes (clearance 0.2))
     (min_thickness 0.2) (filled_areas_thickness no)
@@
     )
   )
-  (zone (net 3) (net_name "/L2-3") (layers "F.Cu" "In1.Cu" "In2.Cu" "In3.Cu" "In4.Cu" "B.Cu") (hatch edge 0.508)
+  (zone (net 3) (net_name "/L2-3") (layers F&B.Cu) (hatch edge 0.508)
     (connect_pads yes (clearance 0.2))
     (min_thickness 0.2) (filled_areas_thickness no)
@@
     )
   )
-  (zone (net 10) (net_name "/L9-10") (layers "F.Cu" "In1.Cu" "In2.Cu" "In3.Cu" "In4.Cu") (hatch edge 0.508)
+  (zone (net 10) (net_name "/L9-10") (layer "F.Cu") (hatch edge 0.508)
     (connect_pads yes (clearance 0.2))
     (min_thickness 0.2) (filled_areas_thickness no)
@@
     )
   )
-  (zone (net 6) (net_name "/L5-6") (layers "F.Cu" "In1.Cu" "In2.Cu" "In3.Cu" "In4.Cu" "B.Cu") (hatch edge 0.508)
+  (zone (net 6) (net_name "/L5-6") (layers F&B.Cu) (hatch edge 0.508)
     (connect_pads yes (clearance 0.2))
     (min_thickness 0.2) (filled_areas_thickness no)
@@
     )
   )
-  (zone (net 7) (net_name "/L6-7") (layers "F.Cu" "In1.Cu" "In2.Cu" "In3.Cu" "In4.Cu" "B.Cu") (hatch edge 0.508)
+  (zone (net 7) (net_name "/L6-7") (layers F&B.Cu) (hatch edge 0.508)
     (connect_pads yes (clearance 0.2))
     (min_thickness 0.2) (filled_areas_thickness no)
@@
     )
   )
-  (zone (net 1) (net_name "/L1A") (layers "F.Cu" "In1.Cu" "In2.Cu" "In3.Cu" "In4.Cu") (hatch edge 0.508)
+  (zone (net 1) (net_name "/L1A") (layer "F.Cu") (hatch edge 0.508)
     (connect_pads yes (clearance 0.2))
     (min_thickness 0.2) (filled_areas_thickness no)
@@
     )
   )
-  (zone (net 5) (net_name "/L4-5") (layers "F.Cu" "In1.Cu" "In2.Cu" "In3.Cu" "In4.Cu" "B.Cu") (hatch edge 0.508)
+  (zone (net 5) (net_name "/L4-5") (layers F&B.Cu) (hatch edge 0.508)
     (connect_pads yes (clearance 0.2))
     (min_thickness 0.2) (filled_areas_thickness no)
@@
     )
   )
-  (zone (net 2) (net_name "/L1-2") (layers "F.Cu" "In1.Cu" "In2.Cu" "In3.Cu" "In4.Cu" "B.Cu") (hatch edge 0.508)
+  (zone (net 2) (net_name "/L1-2") (layers F&B.Cu) (hatch edge 0.508)
     (connect_pads yes (clearance 0.2))
     (min_thickness 0.2) (filled_areas_thickness no)
@@
     )
   )
-  (zone (net 11) (net_name "/L10C") (layers "F.Cu" "In1.Cu" "In2.Cu" "In3.Cu" "In4.Cu" "B.Cu") (hatch edge 0.508)
-    (connect_pads yes (clearance 0.2))
-    (min_thickness 0.2) (filled_areas_thickness no)
+  (zone (net 11) (net_name "/L10C") (layers F&B.Cu) (hatch edge 0.508)
+    (connect_pads yes (clearance 0.2))
+    (min_thickness 0.2) (filled_areas_thickness no)
