File: KiCadProject/StencilTogether/Stencil.kicad_pcb (KiCad board)
At the start: 6 copper layers, 91.9 x 92.1 mm, 216 parts, among them J1 XT30, J101 JST_SM04B, J101 USB-C-2.0, J102 JST_SM04B, J102 Power connector, J103 Data connector, J104 CC connector, J2 XT30, J201 Conn_02x05, J201 USB-C-2.0, J202 Conn_01x02, J202 XT30, J203 Conn_02x05, J204 JST_SM04B, J204 XT60, J205 Conn_02x05, J205 DNP, J206 1x05 female, J206 Conn_01x02_Male, J207 Conn_01x05_Male, J207 JST_SM04B, J208 JST_B5B_XH, J209 Optional off board USB power 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, J210 Optional off board USB CC con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, J3 JST_SM04B, J4 JST_SM04B, Q1 Q_NMOS_GDS, Q2 SUD50P10-43L-GE3, Q301 NFET_Gatenames, Q302 NFET_Gatenames, Q303 NFET_Gatenames, Q304 NFET_Gatenames, Q305 PMOS_Gatenames, Q401 NFET_Gatenames, Q402 PMOS_Gatenames, Q403 NFET_Gatenames, Q404 PMOS_Gatenames, Q405 NFET_Gatenames, Q406 PMOS_Gatenames, Q407 NFET_Gatenames, Q408 PMOS_Gatenames, SW301 SW_Push, SW302 SW_Push, U1 MAX16833, U101 TLE493D, U301 BQ25713, U301 ESP32-S3-WROOM-1, U401 AP63205WU, U402 SC189, U501 PTN5150

Commit message: Started work on body 3d work
Signed-off-by: Eldalote.Electronics <Eldalote.Electronics@gmail.com>
Parts:
- removed the C301 at (128.1, 68.8)
- removed the C301 at (193.8, 78.8)
- removed the C302 at (123.6, 67.8)
- removed the C302 at (193.8, 80.8)
- removed the C303 at (120.0, 67.1)
- removed the C303 at (193.8, 82.8)
- removed the C304 at (149.9, 85.2)
- removed the C304 at (193.8, 84.8)
- removed the C402 at (169.7, 87.5)
- removed the C402 at (122.1, 74.3)
- removed the C403 at (166.8, 92.5)
- removed the C403 at (118.3, 71.0)
- removed the C404 at (166.1, 87.5)
- removed the C404 at (122.1, 71.0)
- removed the D1 at (140.0, 130.5)
- removed the D401 at (118.3, 74.3)
- removed the D401 at (160.8, 85.7)
- removed the J1 at (115.7, 126.2)
- removed the J101 at (183.3, 134.2)
- removed the J101 at (191.3, 117.9)
- removed the J102 at (182.9, 130.8)
- removed the J102 at (175.3, 117.9)
- removed the J201 at (193.8, 90.8)
- removed the J201 at (153.2, 81.0)
- removed the J202 at (166.8, 68.3)
- removed the J202 at (141.3, 91.0)
- removed the J203 at (199.7, 80.8)
- removed the J203 at (115.4, 81.0)
- removed the J204 at (129.3, 97.2)
- removed the J204 at (177.8, 96.3)
- removed the J205 at (119.9, 91.5)
- removed the J205 at (161.8, 80.8)
- removed the J206 at (187.8, 90.8)
- removed the J206 at (134.3, 69.5)
- removed the J207 at (180.8, 69.3)
- removed the J207 at (139.3, 97.2)
- removed the R301 at (121.4, 67.7)
- removed the R301 at (190.8, 77.3)
- removed the R302 at (154.7, 85.3)
- removed the R302 at (188.5, 78.8)
- removed the R303 at (138.3, 91.6)
- removed the R303 at (189.0, 76.8)
- removed the R304 at (138.3, 90.4)
- removed the R304 at (175.1, 90.3)
- removed the R305 at (173.7, 88.2)
- removed the R305 at (139.6, 81.3)
- removed the R306 at (176.6, 88.2)
- removed the R306 at (131.8, 81.3)
- removed the R307 at (187.9, 87.2)
- removed the R307 at (128.3, 81.3)
- removed the R308 at (184.1, 84.0)
- removed the R308 at (123.8, 90.5)
- removed the R309 at (126.8, 90.5)
- removed the R309 at (177.1, 84.3)
- removed the R310 at (129.8, 90.5)
- removed the R310 at (184.5, 88.1)
- removed the R311 at (177.1, 85.3)
- removed the R311 at (132.8, 90.5)
- removed the R312 at (135.8, 90.5)
- removed the R312 at (185.5, 89.1)
- removed the R313 at (138.8, 90.5)
- removed the R313 at (160.4, 81.5)
- removed the R314 at (180.9, 87.7)
- removed the R314 at (141.8, 90.5)
- removed the R315 at (177.1, 86.7)
- removed the R315 at (138.6, 81.3)
- removed the R316 at (197.1, 80.3)
- removed the R316 at (130.8, 81.3)
- removed the R317 at (159.3, 81.5)
- removed the R317 at (127.3, 81.3)
- removed the R318 at (182.6, 88.0)
- removed the R318 at (141.3, 82.0)
- removed the R401 at (163.2, 85.7)
- removed the R401 at (152.6, 71.5)
- removed the REF** at (152.8, 134.4)
- removed the REF** at (169.3, 118.2)
- removed the REF** at (197.3, 117.9)
- removed the REF** at (133.8, 107.9)
- removed the U301 at (134.3, 73.3)
- removed the U301 at (180.8, 83.6)
- added C301: 10u, Capacitor_SMD:C_0805_2012Metric, B.Cu at (131.9, 43.4)
- added C301: 10u, Capacitor_SMD:C_0805_2012Metric, B.Cu at (95.5, 52.8)
- added C302: 100n, Capacitor_SMD:C_0402_1005Metric, F.Cu at (127.5, 42.4)
- added C302: 10u, Capacitor_SMD:C_0805_2012Metric, B.Cu at (95.5, 54.8)
- added C303: 1u, Capacitor_SMD:C_0603_1608Metric, F.Cu at (123.8, 41.7)
- added C303: 10u, Capacitor_SMD:C_0805_2012Metric, B.Cu at (95.5, 56.8)
- added C304: 100n, Capacitor_SMD:C_0402_1005Metric, F.Cu at (153.8, 59.8)
- added C304: 10u, Capacitor_SMD:C_0805_2012Metric, B.Cu at (95.5, 58.8)
- added C402: 10u, Capacitor_SMD:C_0805_2012Metric, F.Cu at (71.4, 61.5)
- added C402: 1u, Capacitor_SMD:C_0603_1608Metric, B.Cu at (126.0, 48.9)
- added C403: 100n, Capacitor_SMD:C_0402_1005Metric, F.Cu at (68.5, 66.3)
- added C403: 1u, Capacitor_SMD:C_0603_1608Metric, B.Cu at (122.2, 45.6)
- added C404: 22u, Capacitor_SMD:C_0805_2012Metric, F.Cu at (67.8, 61.5)
- added C404: 1u, Capacitor_SMD:C_0603_1608Metric, B.Cu at (126.0, 45.6)
- added D1: D_Schottky, Diode_SMD:D_PowerDI-5, F.Cu at (88.9, 108.7)
- added D1: SPHWH1L5N607YEQ3A2, Eldalote-footprints:LED5050_Samsung_LH502C, F.Cu at (142.9, 96.4)
- added D10: SPHWH1L5N607YEQ3A2, Eldalote-footprints:LED5050_Samsung_LH502C, F.Cu at (139.4, 105.8)
- added D2: SPHWH1L5N607YEQ3A2, Eldalote-footprints:LED5050_Samsung_LH502C, F.Cu at (148.1, 100.9)
- added D3: SPHWH1L5N607YEQ3A2, Eldalote-footprints:LED5050_Samsung_LH502C, F.Cu at (149.2, 107.6)
- added D4: SPHWH1L5N607YEQ3A2, Eldalote-footprints:LED5050_Samsung_LH502C, F.Cu at (145.8, 113.5)
- added D401: 3v3, Diode_SMD:D_SOD-523, F.Cu at (122.2, 48.9)
- added D401: GREEN LED, LED_SMD:LED_0805_2012Metric, F.Cu at (62.6, 59.5)
- added D5: SPHWH1L5N607YEQ3A2, Eldalote-footprints:LED5050_Samsung_LH502C, F.Cu at (139.4, 115.8)
- added D6: SPHWH1L5N607YEQ3A2, Eldalote-footprints:LED5050_Samsung_LH502C, F.Cu at (133.0, 113.5)
- added D7: SPHWH1L5N607YEQ3A2, Eldalote-footprints:LED5050_Samsung_LH502C, F.Cu at (129.6, 107.6)
- added D8: SPHWH1L5N607YEQ3A2, Eldalote-footprints:LED5050_Samsung_LH502C, F.Cu at (130.8, 100.8)
- added D9: SPHWH1L5N607YEQ3A2, Eldalote-footprints:LED5050_Samsung_LH502C, F.Cu at (136.0, 96.4)
- added J1: XT30, Eldalote-footprints:XT30, F.Cu at (64.6, 104.4)
- added J1: XT30, Eldalote-footprints:XT30, B.Cu at (139.4, 87.8)
- added J101: USB-C-2.0, Imported:MOLEX_2130830005, F.Cu at (176.7, 105.5)
- added J101: JST_SM04B, Connector_JST:JST_SH_SM04B-SRSS-TB_1x04-1MP_P1.00mm_Horizontal, B.Cu at (177.5, 48.3)
- added J102: JST_SM04B, Connector_JST:JST_SH_SM04B-SRSS-TB_1x04-1MP_P1.00mm_Horizontal, B.Cu at (177.5, 64.3)
- added J102: Power connector, Connector_PinHeader_2.54mm:PinHeader_1x02_P2.54mm_Vertical, B.Cu at (175.4, 102.1)
- added J201: USB-C-2.0, Imported:GCT_USB4120-03-C_REVA, F.Cu at (95.5, 64.8)
- added J201: Conn_02x05, Connector_PinSocket_1.27mm:PinSocket_2x05_P1.27mm_Vertical_SMD, B.Cu at (157.1, 55.6)
- added J202: Conn_01x02, Connector_PinSocket_1.27mm:PinSocket_1x02_P1.27mm_Vertical_SMD_Pin1Left, B.Cu at (145.2, 65.6)
- added J202: XT30, Eldalote-footprints:XT30, B.Cu at (68.5, 42.2)
- added J203: Conn_02x05, Connector_PinHeader_1.27mm:PinHeader_2x05_P1.27mm_Vertical_SMD, F.Cu at (101.4, 54.8)
- added J203: Conn_02x05, Connector_PinSocket_1.27mm:PinSocket_2x05_P1.27mm_Vertical_SMD, B.Cu at (119.3, 55.6)
- added J204: XT60, Eldalote-footprints:XT60, B.Cu at (79.5, 70.2)
- added J204: JST_SM04B, Connector_JST:JST_SH_SM04B-SRSS-TB_1x04-1MP_P1.00mm_Horizontal, B.Cu at (133.2, 71.8)
- added J205: DNP, Connector_PinHeader_1.27mm:PinHeader_2x02_P1.27mm_Vertical_SMD, F.Cu at (123.8, 66.0)
- added J205: Conn_02x05, Connector_PinHeader_1.27mm:PinHeader_2x05_P1.27mm_Vertical_SMD, F.Cu at (63.6, 54.8)
- added J206: Conn_01x02_Male, Connector_PinHeader_1.27mm:PinHeader_1x02_P1.27mm_Vertical_SMD_Pin1Left, F.Cu at (89.5, 64.8)
- added J206: 1x05 female, Connector_PinSocket_1.27mm:PinSocket_1x05_P1.27mm_Vertical_SMD_Pin1Left, B.Cu at (138.2, 44.1)
- added J207: Conn_01x05_Male, Connector_PinHeader_1.27mm:PinHeader_1x05_P1.27mm_Vertical_SMD_Pin1Left, F.Cu at (82.5, 43.2)
- added J207: JST_SM04B, Connector_JST:JST_SH_SM04B-SRSS-TB_1x04-1MP_P1.00mm_Horizontal, B.Cu at (143.2, 71.8)
- added R301: 10k, Resistor_SMD:R_0402_1005Metric, F.Cu at (125.3, 42.2)
- added R301: 10m, Resistor_SMD:R_1206_3216Metric, B.Cu at (92.5, 51.2)
- added R302: 100k, Resistor_SMD:R_0402_1005Metric, F.Cu at (158.6, 59.9)
- added R302: 4R99, Resistor_SMD:R_0402_1005Metric, B.Cu at (90.2, 52.8)
- added R303: 4R99, Resistor_SMD:R_0402_1005Metric, B.Cu at (90.8, 50.8)
- added R303: JMP, Resistor_SMD:R_0402_1005Metric, B.Cu at (142.2, 66.2)
- added R304: 10m, Resistor_SMD:R_1206_3216Metric, B.Cu at (76.8, 64.2)
- added R304: JMP, Resistor_SMD:R_0402_1005Metric, B.Cu at (142.2, 65.0)
- added R305: 10R, Resistor_SMD:R_0402_1005Metric, B.Cu at (75.4, 62.1)
- added R305: 100k, Resistor_SMD:R_0402_1005Metric, B.Cu at (143.4, 55.9)
- added R306: 10R, Resistor_SMD:R_0402_1005Metric, B.Cu at (78.3, 62.0)
- added R306: 100k, Resistor_SMD:R_0402_1005Metric, B.Cu at (140.5, 55.9)
- added R307: 100k, Resistor_SMD:R_0402_1005Metric, B.Cu at (137.7, 55.9)
- added R307: 1R, Resistor_SMD:R_0603_1608Metric, B.Cu at (89.7, 61.0)
- added R308: 240R, Resistor_SMD:R_0402_1005Metric, F.Cu at (127.7, 65.1)
- added R308: 10R, Resistor_SMD:R_0402_1005Metric, F.Cu at (85.8, 58.0)
- added R309: 240R, Resistor_SMD:R_0402_1005Metric, F.Cu at (130.7, 65.1)
- added R309: 100k, Resistor_SMD:R_0402_1005Metric, F.Cu at (78.8, 58.2)
- added R310: 240R, Resistor_SMD:R_0402_1005Metric, F.Cu at (133.7, 65.1)
- added R310: 174k, Resistor_SMD:R_0402_1005Metric, B.Cu at (86.2, 62.0)
- added R311: 240R, Resistor_SMD:R_0402_1005Metric, F.Cu at (136.7, 65.1)
- added R311: 300k, Resistor_SMD:R_0402_1005Metric, F.Cu at (78.8, 59.2)
- added R312: 240R, Resistor_SMD:R_0402_1005Metric, F.Cu at (139.7, 65.1)
- added R312: 100k, Resistor_SMD:R_0402_1005Metric, B.Cu at (87.2, 63.0)
- added R313: 240R, Resistor_SMD:R_0402_1005Metric, F.Cu at (142.7, 65.1)
- added R313: 100k, Resistor_SMD:R_0402_1005Metric, B.Cu at (62.2, 55.5)
- added R314: 240R, Resistor_SMD:R_0402_1005Metric, F.Cu at (145.7, 65.1)
- added R314: 40K2, Resistor_SMD:R_0402_1005Metric, F.Cu at (82.7, 61.5)
- added R315: 10k, Resistor_SMD:R_0402_1005Metric, F.Cu at (78.8, 60.5)
- added R315: DNP, Resistor_SMD:R_0402_1005Metric, B.Cu at (142.4, 55.9)
- added R316: DNP, Resistor_SMD:R_0402_1005Metric, B.Cu at (139.5, 55.9)
- added R316: 10k, Resistor_SMD:R_0402_1005Metric, B.Cu at (98.8, 54.2)
- added R317: DNP, Resistor_SMD:R_0402_1005Metric, B.Cu at (136.7, 55.9)
- added R317: 10k, Resistor_SMD:R_0402_1005Metric, B.Cu at (61.1, 55.5)
- added R318: 137k, Resistor_SMD:R_0402_1005Metric, B.Cu at (84.3, 62.0)
- added R318: 5k1, Resistor_SMD:R_0402_1005Metric, B.Cu at (145.2, 56.6)
- added R401: 649R, Resistor_SMD:R_0402_1005Metric, F.Cu at (64.9, 59.5)
- added R401: 10k, Resistor_SMD:R_0402_1005Metric, B.Cu at (156.5, 46.1)
- added REF**: MountingHole_2.2mm_M2, MountingHole:MountingHole_2.2mm_M2, F.Cu at (177.5, 42.3)
- added REF**: MountingHole_2.2mm_M2, MountingHole:MountingHole_2.2mm_M2, F.Cu at (122.4, 105.8)
- added REF**: MountingHole_2.2mm_M2, MountingHole:MountingHole_2.2mm_M2, F.Cu at (156.4, 105.8)
- added REF**: MountingHole_2.2mm_M2, MountingHole:MountingHole_2.2mm_M2, F.Cu at (82.7, 86.1)
- added REF**: MountingHole_2.2mm_M2, MountingHole:MountingHole_2.2mm_M2, F.Cu at (177.8, 70.3)
- added REF**: MountingHole_2.2mm_M2, MountingHole:MountingHole_2.2mm_M2, F.Cu at (101.7, 112.6)
- added REF**: MountingHole_2.2mm_M2, MountingHole:MountingHole_2.2mm_M2, F.Cu at (139.4, 122.8)
- added U301: ESP32-S3-WROOM-1, Imported:XCVR_ESP32-S3-WROOM-1, F.Cu at (138.2, 47.9)
- added U301: BQ25713, Package_DFN_QFN:Texas_S-PWQFN-N32_EP2.8x2.8mm, B.Cu at (82.5, 57.5)
- moved C330 101.7 mm to (78.8, 61.5)
- moved C407 101.7 mm to (64.8, 59.0)
- moved L401 101.7 mm to (66.3, 64.0)
- moved C305 101.7 mm to (89.5, 59.2)
- moved C306 101.7 mm to (89.5, 57.2)
- moved C307 101.7 mm to (89.5, 55.2)
- moved C308 101.7 mm to (89.2, 53.8)
- moved C309 101.7 mm to (89.5, 50.8)
- moved C310 101.7 mm to (94.8, 48.0)
- moved C311 101.7 mm to (94.8, 49.0)
- moved C312 101.7 mm to (84.0, 54.0)
- moved C313 101.7 mm to (80.0, 54.0)
- moved C314 101.7 mm to (69.3, 51.8)
- moved C315 101.7 mm to (69.3, 57.8)
- moved C316 101.7 mm to (69.3, 55.8)
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Routing:
- net (no net): track 2072.4 -> 2076.5 mm, vias 657 -> 698
- added copper zone on In1.Cu, net (none)
Other:
- board size 91.9 x 92.1 mm -> 123.2 x 96.3 mm
- board text added: "Hi, my name is Jacob"
- board text added: "Led Board"
